Commit message: renaming

File: hagen_robot/hagen_description/urdf/base/forklift_base.urdf.xacro (robot description, xacro)
@@ -1,4 +1,4 @@
 <?xml version="1.0"?>
-<!-- Dyno Magni base -->
+<!-- hagen Magni base -->
 <robot xmlns:xacro="http://ros.org/wiki/xacro">
   <xacro:include filename="forklift_base.gazebo.xacro"/>
@@ -11,5 +11,5 @@
         <origin xyz="0 0 0" rpy="0 0 0"/>
         <geometry>
-          <mesh filename="package://dyno_description/meshes/bases/forklift_base.stl" scale="0.01 0.01 0.01"/>
+          <mesh filename="package://hagen_description/meshes/bases/forklift_base.stl" scale="0.01 0.01 0.01"/>
         </geometry>
         <material name="dark"/>
@@ -48,5 +48,5 @@
         <origin xyz="0 0 0" rpy="0 0 ${M_PI}"/>
         <geometry>
-          <mesh filename="package://dyno_description/meshes/bases/forklift_fork.stl" scale="0.01 0.01 0.01"/>
+          <mesh filename="package://hagen_description/meshes/bases/forklift_fork.stl" scale="0.01 0.01 0.01"/>
         </geometry>
         <material name="black"/>

File: hagen_robot/hagen_description/urdf/base/magni_base.urdf.xacro (robot description, xacro)
@@ -1,4 +1,4 @@
 <?xml version="1.0"?>
-<!-- Dyno Magni base -->
+<!-- hagen Magni base -->
 <robot xmlns:xacro="http://ros.org/wiki/xacro">
   <xacro:include filename="magni_base.gazebo.xacro"/>

File: hagen_robot/hagen_description/urdf/base/magni_sign_base.urdf.xacro (robot description, xacro)
@@ -1,4 +1,4 @@
 <?xml version="1.0"?>
-<!-- Dyno Magni base -->
+<!-- hagen Magni base -->
 <robot xmlns:xacro="http://ros.org/wiki/xacro">
   <xacro:include filename="magni_sign_base.gazebo.xacro"/>
@@ -21,5 +21,5 @@
         <geometry>
           <!-- <box size="${wheel_separation*1.3} ${wheel_separation-wheel_width} 0.25"/> -->
-          <mesh filename="package://dyno_description/meshes/bases/magni_sign_base.dae" scale="0.01 0.01 0.01"/>
+          <mesh filename="package://hagen_description/meshes/bases/magni_sign_base.dae" scale="0.01 0.01 0.01"/>
         </geometry>
       </visual>
@@ -52,5 +52,5 @@
         <origin xyz="0 0 0" rpy="0 0 0"/>
         <geometry>
-          <mesh filename="package://dyno_description/meshes/other/sign_pole.stl" scale="0.01 0.01 0.01"/>
+          <mesh filename="package://hagen_description/meshes/other/sign_pole.stl" scale="0.01 0.01 0.01"/>
         </geometry>
         <material name="grey"/>
@@ -67,5 +67,5 @@
         <origin xyz="0 0 0" rpy="0 0 0"/>
         <geometry>
-          <mesh filename="package://dyno_description/meshes/other/monitor_43.dae" scale="0.01 0.01 0.01"/>
+          <mesh filename="package://hagen_description/meshes/other/monitor_43.dae" scale="0.01 0.01 0.01"/>
         </geometry>
         <material name="black"/>

File: hagen_robot/hagen_description/urdf/base/omnibot_base.urdf.xacro (robot description, xacro)
@@ -1,4 +1,4 @@
 <?xml version="1.0"?>
-<!-- Dyno differential mecanum base -->
+<!-- hagen differential mecanum base -->
 <robot xmlns:xacro="http://ros.org/wiki/xacro">
   <xacro:include filename="omnibot_base.gazebo.xacro"/>
@@ -13,5 +13,5 @@
         <origin xyz="0 0 0.02" rpy="0 0 0"/>
         <geometry>
-          <mesh filename="package://dyno_description/meshes/bases/omnibot_base.stl" scale="0.001 0.001 0.001"/>
+          <mesh filename="package://hagen_description/meshes/bases/omnibot_base.stl" scale="0.001 0.001 0.001"/>
         </geometry>
         <material name="light_blue"/>

File: hagen_robot/hagen_description/urdf/base/quadrotor_base.urdf.xacro (robot description, xacro)
@@ -13,5 +13,5 @@
         <origin xyz="0 0 0" rpy="0 0 0"/>
         <geometry>
-          <mesh filename="package://dyno_description/meshes/quadrotor/quadrotor_base.dae"/>
+          <mesh filename="package://hagen_description/meshes/quadrotor/quadrotor_base.dae"/>
         </geometry>
       </visual>
@@ -19,5 +19,5 @@
         <origin xyz="0 0 0" rpy="0 0 0"/>
         <geometry>
-          <mesh filename="package://dyno_description/meshes/quadrotor/quadrotor_base.stl"/>
+          <mesh filename="package://hagen_description/meshes/quadrotor/quadrotor_base.stl"/>
         </geometry>
       </collision>

File: hagen_robot/hagen_description/urdf/base/turtlebot3_burger.urdf.xacro (robot description, xacro)
@@ -1,4 +1,4 @@
 <?xml version="1.0" ?>
-<!-- Dyno turtlebot3 base -->
+<!-- hagen turtlebot3 base -->
 <robot xmlns:xacro="http://ros.org/wiki/xacro">
   <xacro:include filename="turtlebot3_burger.gazebo.xacro"/>
@@ -16,5 +16,5 @@
         <origin xyz="-0.032 0 0.0" rpy="0 0 0"/>
         <geometry>
-          <mesh filename="package://dyno_description/meshes/bases/burger_base.stl" scale="0.001 0.001 0.001"/>
+          <mesh filename="package://hagen_description/meshes/bases/burger_base.stl" scale="0.001 0.001 0.001"/>
         </geometry>
         <material name="light_black"/>

File: hagen_robot/hagen_description/urdf/hagen.urdf.xacro (robot description, xacro)
@@ -139,5 +139,5 @@
       <origin xyz="${forklift_x_offset} ${forklift_y_offset} ${forklift_z_offset}" rpy="0 0 0"/>
       <geometry>
-        <mesh filename="package://dyno_description/meshes/bases/forklift_base.stl" scale="0.03 0.03 0.01"/>
+        <mesh filename="package://hagen_description/meshes/bases/forklift_base.stl" scale="0.03 0.03 0.01"/>
       </geometry>
       <material name="dark"/>
@@ -171,5 +171,5 @@
       <origin xyz="${forkjoint_x_offset} ${forklift_y_offset} ${forklift_z_offset}" rpy="0 0 ${PI}"/>
       <geometry>
-        <mesh filename="package://dyno_description/meshes/bases/forklift_fork.stl" scale="0.02 0.03 0.01"/>
+        <mesh filename="package://hagen_description/meshes/bases/forklift_fork.stl" scale="0.02 0.03 0.01"/>
       </geometry>
       <material name="black"/>

File: hagen_robot/hagen_description/urdf/manipulators/open_manipulator.urdf.xacro (robot description, xacro)
@@ -3,5 +3,5 @@
 <robot xmlns:xacro="http://www.ros.org/wiki/xacro">
   <!-- Include OpenManipulator Chain Gazebo Parameter -->
-  <xacro:include filename="$(find dyno_description)/urdf/manipulators/open_manipulator.gazebo.xacro"/>
+  <xacro:include filename="$(find hagen_description)/urdf/manipulators/open_manipulator.gazebo.xacro"/>
   <xacro:macro name="open_manipulator" params="x_offset y_offset z_offset">
     <!-- Base fixed joint -->
@@ -16,12 +16,12 @@
         <origin xyz="0 0 0" rpy="0 0 0"/>
         <geometry>
-          <mesh filename="package://dyno_description/meshes/manipulators/open_manipulator/chain_link1.stl" scale="0.001 0.001 0.001"/>
-        </geometry>
-        <material name="dark"/>
-      </visual>
-      <collision>
-        <origin xyz="0 0 0" rpy="0 0 0"/>
-        <geometry>
-          <mesh filename="package://dyno_description/meshes/manipulators/open_manipulator/chain_link1.stl" scale="0.001 0.001 0.001"/>
+          <mesh filename="package://hagen_description/meshes/manipulators/open_manipulator/chain_link1.stl" scale="0.001 0.001 0.001"/>
+        </geometry>
+        <material name="dark"/>
+      </visual>
+      <collision>
+        <origin xyz="0 0 0" rpy="0 0 0"/>
+        <geometry>
+          <mesh filename="package://hagen_description/meshes/manipulators/open_manipulator/chain_link1.stl" scale="0.001 0.001 0.001"/>
         </geometry>
       </collision>
@@ -57,5 +57,5 @@
         <origin xyz="0 0 0.018" rpy="0 0 0"/>
         <geometry>
-          <mesh filename="package://dyno_description/meshes/manipulators/open_manipulator/chain_link2.stl" scale="0.001 0.001 0.001"/>
+          <mesh filename="package://hagen_description/meshes/manipulators/open_manipulator/chain_link2.stl" scale="0.001 0.001 0.001"/>
         </geometry>
         <material name="dark"/>
@@ -64,5 +64,5 @@
         <origin xyz="0 0 0.018" rpy="0 0 0"/>
         <geometry>
-          <mesh filename="package://dyno_description/meshes/manipulators/open_manipulator/chain_link2.stl" scale="0.001 0.001 0.001"/>
+          <mesh filename="package://hagen_description/meshes/manipulators/open_manipulator/chain_link2.stl" scale="0.001 0.001 0.001"/>
         </geometry>
       </collision>
@@ -99,12 +99,12 @@
         <origin xyz="0 0 0" rpy="0 0 0"/>
         <geometry>
-          <mesh filename="package://dyno_description/meshes/manipulators/open_manipulator/chain_link3.stl" scale="0.001 0.001 0.001"/>
-        </geometry>
-        <material name="dark"/>
-      </visual>
-      <collision>
-        <origin xyz="0 0 0" rpy="0 0 0"/>
-        <geometry>
-          <mesh filename="package://dyno_description/meshes/manipulators/open_manipulator/chain_link3.stl" scale="0.001 0.001 0.001"/>
+          <mesh filename="package://hagen_description/meshes/manipulators/open_manipulator/chain_link3.stl" scale="0.001 0.001 0.001"/>
+        </geometry>
+        <material name="dark"/>
+      </visual>
+      <collision>
+        <origin xyz="0 0 0" rpy="0 0 0"/>
+        <geometry>
+          <mesh filename="package://hagen_description/meshes/manipulators/open_manipulator/chain_link3.stl" scale="0.001 0.001 0.001"/>
         </geometry>
       </collision>
@@ -141,12 +141,12 @@
         <origin xyz="0 0 0" rpy="0 0 0"/>
         <geometry>
-          <mesh filename="package://dyno_description/meshes/manipulators/open_manipulator/chain_link4.stl" scale="0.001 0.001 0.001"/>
-        </geometry>
-        <material name="dark"/>
-      </visual>
-      <collision>
-        <origin xyz="0 0 0" rpy="0 0 0"/>
-        <geometry>
-          <mesh filename="package://dyno_description/meshes/manipulators/open_manipulator/chain_link4.stl" scale="0.001 0.001 0.001"/>
+          <mesh filename="package://hagen_description/meshes/manipulators/open_manipulator/chain_link4.stl" scale="0.001 0.001 0.001"/>
+        </geometry>
+        <material name="dark"/>
+      </visual>
+      <collision>
+        <origin xyz="0 0 0" rpy="0 0 0"/>
+        <geometry>
+          <mesh filename="package://hagen_description/meshes/manipulators/open_manipulator/chain_link4.stl" scale="0.001 0.001 0.001"/>
         </geometry>
       </collision>
@@ -183,12 +183,12 @@
         <origin xyz="0 0 0" rpy="0 0 0"/>
         <geometry>
-          <mesh filename="package://dyno_description/meshes/manipulators/open_manipulator/chain_link5.stl" scale="0.001 0.001 0.001"/>
-        </geometry>
-        <material name="dark"/>
-      </visual>
-      <collision>
-        <origin xyz="0 0 0" rpy="0 0 0"/>
-        <geometry>
-          <mesh filename="package://dyno_description/meshes/manipulators/open_manipulator/chain_link5.stl" scale="0.001 0.001 0.001"/>
+          <mesh filename="package://hagen_description/meshes/manipulators/open_manipulator/chain_link5.stl" scale="0.001 0.001 0.001"/>
+        </geometry>
+        <material name="dark"/>
+      </visual>
+      <collision>
+        <origin xyz="0 0 0" rpy="0 0 0"/>
+        <geometry>
+          <mesh filename="package://hagen_description/meshes/manipulators/open_manipulator/chain_link5.stl" scale="0.001 0.001 0.001"/>
         </geometry>
       </collision>
@@ -205,5 +205,5 @@
         <origin xyz="0.028 0.0246 0" rpy="0 0 0"/>
         <geometry>
-          <mesh filename="package://dyno_description/meshes/manipulators/open_manipulator/chain_link_grip_l.stl" scale="0.001 0.001 0.001"/>
+          <mesh filename="package://hagen_description/meshes/manipulators/open_manipulator/chain_link_grip_l.stl" scale="0.001 0.001 0.001"/>
         </geometry>
         <material name="dark"/>
@@ -212,5 +212,5 @@
         <origin xyz="0.028 0.0246 0" rpy="0 0 0"/>
         <geometry>
-          <mesh filename="package://dyno_description/meshes/manipulators/open_manipulator/chain_link_grip_l.stl" scale="0.001 0.001 0.001"/>
+          <mesh filename="package://hagen_description/meshes/manipulators/open_manipulator/chain_link_grip_l.stl" scale="0.001 0.001 0.001"/>
         </geometry>
       </collision>
@@ -247,5 +247,5 @@
         <origin xyz="0.028 -0.0246 0" rpy="0 0 0"/>
         <geometry>
-          <mesh filename="package://dyno_description/meshes/manipulators/open_manipulator/chain_link_grip_r.stl" scale="0.001 0.001 0.001"/>
+          <mesh filename="package://hagen_description/meshes/manipulators/open_manipulator/chain_link_grip_r.stl" scale="0.001 0.001 0.001"/>
         </geometry>
         <material name="dark"/>
@@ -254,5 +254,5 @@
         <origin xyz="0.028 -0.0246 0" rpy="0 0 0"/>
         <geometry>
-          <mesh filename="package://dyno_description/meshes/manipulators/open_manipulator/chain_link_grip_r.stl" scale="0.001 0.001 0.001"/>
+          <mesh filename="package://hagen_description/meshes/manipulators/open_manipulator/chain_link_grip_r.stl" scale="0.001 0.001 0.001"/>
         </geometry>
       </collision>

File: hagen_robot/hagen_description/urdf/sensors/lds_lfcd.urdf.xacro (robot description, xacro)
@@ -12,5 +12,5 @@
         <origin xyz="0 0 0.0" rpy="0 0 0"/>
         <geometry>
-          <mesh filename="package://dyno_description/meshes/sensors/lds.stl" scale="0.001 0.001 0.001"/>
+          <mesh filename="package://hagen_description/meshes/sensors/lds.stl" scale="0.001 0.001 0.001"/>
           <!-- <cylinder length="0.0315" radius="0.055"/> -->
         </geometry>

File: hagen_robot/hagen_description/urdf/sensors/leap_motion.urdf.xacro (robot description, xacro)
@@ -12,5 +12,5 @@
         <origin xyz="0 0 0.0" rpy="0 0 0"/>
         <geometry>
-          <mesh filename="package://dyno_description/meshes/sensors/leap_motion.dae" scale="0.01 0.01 0.01"/>
+          <mesh filename="package://hagen_description/meshes/sensors/leap_motion.dae" scale="0.01 0.01 0.01"/>
         </geometry>
         <!-- <material name="grey"/> -->

File: hagen_robot/hagen_description/urdf/sensors/rplidar_a2.urdf.xacro (robot description, xacro)
@@ -12,5 +12,5 @@
         <origin xyz="0 0 0.0" rpy="0 0 0"/>
         <geometry>
-          <mesh filename="package://dyno_description/meshes/sensors/rplidar_a2.dae" scale="0.01 0.01 0.01"/>
+          <mesh filename="package://hagen_description/meshes/sensors/rplidar_a2.dae" scale="0.01 0.01 0.01"/>
         </geometry>
       </visual>

File: hagen_robot/hagen_description/urdf/sensors/sick_tim.urdf.xacro (robot description, xacro)
@@ -9,5 +9,5 @@
       min_range="${min_range}" max_range="${max_range}"
       min_angle="${min_angle}" max_angle="${max_angle}"
-      mesh="package://dyno_description/meshes/sensors/sick_tim551.stl" />
+      mesh="package://hagen_description/meshes/sensors/sick_tim551.stl" />
   </xacro:macro>
   <xacro:macro name="sick_tim" params="name ros_topic length width height mass z_offset min_angle max_angle min_range max_range mesh">

File: hagen_robot/hagen_description/urdf/sensors/sonar_sensor.urdf.xacro (robot description, xacro)
@@ -17,5 +17,5 @@
         <geometry>
           <!--<box size="0.01 0.01 0.01" /> -->
-          <mesh filename="package://dyno_description/meshes/sensors/sonar_sensor/max_sonar_ez4.dae"/>
+          <mesh filename="package://hagen_description/meshes/sensors/sonar_sensor/max_sonar_ez4.dae"/>
         </geometry>
       </visual>

File: hagen_robot/hagen_description/urdf/sensors/sweep.urdf.xacro (robot description, xacro)
@@ -6,5 +6,5 @@
       length="0.065" width="0.065" height="0.0619" mass="0.120" z_offset="0.0415"
       min_range="${0.05}" max_range="${15.0}"
-      mesh="package://dyno_description/meshes/sensors/sweep.dae" />
+      mesh="package://hagen_description/meshes/sensors/sweep.dae" />
   </xacro:macro>
   <xacro:macro name="scanse_sweep" params="name ros_topic length width height mass z_offset min_range max_range mesh">

File: hagen_robot/hagen_description/urdf/sensors/vive_tracker.urdf.xacro (robot description, xacro)
@@ -12,5 +12,5 @@
         <origin xyz="0 0 0.0" rpy="0 0 0"/>
         <geometry>
-          <mesh filename="package://dyno_description/meshes/sensors/vive_tracker.stl" scale="0.01 0.01 0.01"/>
+          <mesh filename="package://hagen_description/meshes/sensors/vive_tracker.stl" scale="0.01 0.01 0.01"/>
         </geometry>
         <material name="black"/>

File: hagen_robot/hagen_description/urdf/wheels/forklift/drive_wheel_assembly.urdf.xacro (robot description, xacro)
@@ -30,5 +30,5 @@
       <visual>
         <geometry>
-          <mesh filename="package://dyno_description/meshes/wheels/forklift_drive_wheel.stl" scale="0.01 0.01 0.01"/>
+          <mesh filename="package://hagen_description/meshes/wheels/forklift_drive_wheel.stl" scale="0.01 0.01 0.01"/>
         </geometry>
         <material name="DarkGrey"/>
@@ -61,5 +61,5 @@
         <origin xyz="0 0 0" rpy="0 0 0"/>
         <geometry>
-          <mesh filename="package://dyno_description/meshes/bases/forklift_steer.stl" scale="0.01 0.01 0.01"/>
+          <mesh filename="package://hagen_description/meshes/bases/forklift_steer.stl" scale="0.01 0.01 0.01"/>
         </geometry>
         <material name="light_blue"/>

File: hagen_robot/hagen_description/urdf/wheels/forklift/support_wheel.urdf.xacro (robot description, xacro)
@@ -10,5 +10,5 @@
         <origin xyz="0 0 0" rpy="0 0 0"/>
         <geometry>
-          <mesh filename="package://dyno_description/meshes/wheels/forklift_support_wheel.stl" scale="0.01 0.01 0.01"/>
+          <mesh filename="package://hagen_description/meshes/wheels/forklift_support_wheel.stl" scale="0.01 0.01 0.01"/>
         </geometry>
         <material name="orange"/>

File: hagen_robot/hagen_description/urdf/wheels/magni/drive_wheel.urdf.xacro (robot description, xacro)
@@ -9,5 +9,5 @@
         <geometry>
           <!-- <cylinder radius="${radius}" length="${width}"/> -->
-          <mesh filename="package://dyno_description/meshes/wheels/magni_wheel.dae" scale="0.0118 0.0118 ${-0.0118 * reflect}"/>
+          <mesh filename="package://hagen_description/meshes/wheels/magni_wheel.dae" scale="0.0118 0.0118 ${-0.0118 * reflect}"/>
         </geometry>
       </visual>

File: hagen_robot/hagen_description/urdf/wheels/omnibot/mecanum_wheel.urdf.xacro (robot description, xacro)
@@ -9,8 +9,8 @@
         <geometry>
           <xacro:if value="${type == 'left'}">
-            <mesh filename="package://dyno_description/meshes/wheels/mecanum_wheel.stl" scale="0.001 0.001 0.001"/>
+            <mesh filename="package://hagen_description/meshes/wheels/mecanum_wheel.stl" scale="0.001 0.001 0.001"/>
           </xacro:if>
           <xacro:if value="${type == 'right'}">
-            <mesh filename="package://dyno_description/meshes/wheels/mecanum_wheel.stl" scale="0.001 0.001 -0.001"/>
+            <mesh filename="package://hagen_description/meshes/wheels/mecanum_wheel.stl" scale="0.001 0.001 -0.001"/>
           </xacro:if>
         </geometry>

File: hagen_robot/hagen_description/urdf/wheels/turtlebot3/drive_wheel.urdf.xacro (robot description, xacro)
@@ -8,5 +8,5 @@
         <origin xyz="0 0 0" rpy="${1.57*reflect} 0 0"/>
         <geometry>
-          <mesh filename="package://dyno_description/meshes/wheels/right_tire.stl" scale="0.001 0.001 0.001"/>
+          <mesh filename="package://hagen_description/meshes/wheels/right_tire.stl" scale="0.001 0.001 0.001"/>
         </geometry>
         <material name="dark"/>
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